File: Li-ion 5A Boost 1A Charge Protect/Li-ion 5A Boost 1A Charge Protect.kicad_pcb (KiCad board)
At the start: 2 copper layers, 51.5 x 32 mm, 55 parts, among them J1 USB_C_FEMALE, Q1 BUK6D30-40E, SW1 SW_DPST, U1 AP9101CK6, U2 ECH8695R-TL-W, U3 MCP73833T, U4 PAM2423AECADJR

Commit message: Near complete version 1.1.0
Parts:
- moved W2 7.10 mm to (134.9, 70.2)
- moved H3 6.99 mm to (142.0, 71.8)
- moved W5 4.00 mm to (114.0, 69.9)
- moved F4 3.58 mm to (107.9, 81.1)
- moved F3 3.35 mm to (128.6, 69.7)
- moved C1 3.30 mm to (111.7, 74.9), turned to 90 degrees
- moved H4 2.39 mm to (102.6, 70.6)
- moved R2 2.33 mm to (109.6, 78.7), turned to 270 degrees
- moved U1 2.01 mm to (108.5, 75.2), turned to 0 degrees
- moved W6 2.00 mm to (107.6, 69.9)
- moved U2 1.58 mm to (103.8, 75.2)
- moved R1 1.47 mm to (111.7, 78.7)
- moved R13 1.18 mm to (117.9, 76.5)
- moved R14 1.18 mm to (117.9, 78.3)
- moved Q1 1.01 mm to (104.2, 80.7)
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Connections:
- SW1 pad 2: /BATT+ -> Net-(R13-Pad2)
- SW1 pad 3: Net-(R13-Pad2) -> /BATT+
- SW1 pad 5: /BATT+ -> Net-(R13-Pad2)
- SW1 pad 6: Net-(R13-Pad2) -> /BATT+
Routing:
- net Net-(R13-Pad2): track 5.64 -> 11.3 mm, vias 0 -> 1
- net Net-(Q1-Pad3): track 18.9 -> 15.1 mm
- net /ST1: track 8.26 -> 10.7 mm
- net /PVDD: track 6.62 -> 4.27 mm
- net Net-(U1-Pad3): track 9.55 -> 7.30 mm
- net Net-(U1-Pad1): track 6.78 -> 5.15 mm
- net /PVM: track 2.73 -> 4.26 mm
- net /VUSB: track 5.97 -> 4.49 mm
- net GND: track 17.8 -> 16.6 mm, vias 11 -> 17
- net /THRMIC: track 8.39 -> 7.37 mm
- net /PROG: track 12.4 -> 11.6 mm
- net /ST2: track 7.29 -> 6.75 mm
- net /BATT-: track 0.00 -> 0.53 mm, vias 6 -> 9
- net (no net): track 0.36 -> 0.00 mm, vias 3 -> 0
- net /BATT+: track 3.11 -> 2.88 mm, vias 4 -> 6
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Other:
- net class Default: clearance 0.2 -> 0.1524
- net class High Power: clearance 0.2 -> 0.1524
- rule trace_clearance: 0.2 -> 0.1524
- board text added: "1A Charge"
- board text added: "5V 5.5A Output"
- board text added: "5V OUT"
- board text added: "Li-Ion"
- board text removed: "+ 5V OUT -"
- board text removed: "Li-Ion 5V 5.5A Output 1A Charge"
