File: Li-ion 5A Boost 1A Charge Protect/Li-ion 5A Boost 1A Charge Protect.sch (KiCad schematic (older format))
At the start: 44 parts, among them J1 USB_C_FEMALE, SW1 SW_SPST, U1 AP9101CK6, U2 ECH8695R-TL-W, U3 MCP73833T, U4 PAM2423AECADJR

Commit message: Standarizing libraries
Parts:
- C1, C10, C2, C4, C5, C6, C7, C8, C9: symbol Li-ion_LE:C -> Frequently_Used_LE:C
- C11, C3: symbol Li-ion_LE:CP1 -> Frequently_Used_LE:CP1
- L1: symbol Li-ion_LE:L -> Frequently_Used_LE:L
- LD1, LD2, LD3, LD4: symbol Li-ion_LE:LED -> Frequently_Used_LE:LED
- R1, R10, R11, R12, R2, R3, R4, R5, R6, R7, R8, R9: symbol Li-ion_LE:R -> Frequently_Used_LE:R
- SW1: symbol Li-ion_LE:SW_SPST -> Frequently_Used_LE:SW_SPST
- TH1: symbol Li-ion_LE:Thermistor_NTC -> Li_Ion_LE:Thermistor_NTC
- U1: symbol Li-ion_LE:AP9101CK6 -> Li_Ion_LE:AP9101CK6
- U2: symbol Li-ion_LE:ECH8695R-TL-W_Gates_on_Top -> Li_Ion_LE:ECH8695R-TL-W_Gates_on_Top
- U3: symbol Li-ion_LE:MCP73833T -> Li_Ion_LE:MCP73833T
- U4: symbol Li-ion_LE:PAM2423AECADJR -> Li_Ion_LE:PAM2423AECADJR
- W1, W2, W3, W4, W5, W6, W7, W8: symbol Li-ion_LE:TestPoint -> Frequently_Used_LE:TestPoint_1

Commit message: Library updates
Parts:
- added FID1, FID2, FID3: Fiducial, Fiducial_LE:Fiducial_1mm_Mask2mm, symbol Mechanical_LE:Fiducial
- C1: value 100nF -> 0.1uF; footprint Li-ion:0805_2012Metric_HandSolder -> Frequently_Used_LE:0805_2012Metric_HandSolder
- C10, C2, C4, C5, C6, C7, C8, C9, R1, R10, R11, R12, R2, R3, R4, R5, R6, R7, R8, R9, TH1: footprint Li-ion:0805_2012Metric_HandSolder -> Frequently_Used_LE:0805_2012Metric_HandSolder
- C11, C3: footprint Li-ion:UCD1E471MNL1GS -> Li_Ion_LE:25TLV470M10X10.5; Manufacturer Name Nichicon -> Rubycon; Manufacturer Part No. UCD1E471MNL1GS -> 25TLV470M10X10.5; Source Part No. 493-6386-1-ND -> 1189-2097-1-ND
- D1: footprint Li-ion:NTS12120EMFST1G -> Li_Ion_LE:NTS12120EMFST1G; symbol Li-ion_LE:D_NTS12120EMFST1G -> Li_Ion_LE:D_NTS12120EMFST1G
- J1: footprint Li-ion:GCT_USB4110-GF-A -> Connector_LE:GCT_USB4110-GF-A; symbol Connectors_LE:USB_C_Plug_USB2.0 -> Connector_LE:USB_C_Plug_USB2.0
- L1: footprint Li-ion:L_MGV1004 -> Li_Ion_LE:L_MGV1004
- LD1, LD2, LD3, LD4: footprint Li-ion:LED_0805_2012Metric_HandSolder -> Li_Ion_LE:LED_0805_2012Metric_HandSolder
- SW1: footprint Li-ion:GF1230054 -> Li_Ion_LE:GF1230054
- U1: footprint Li-ion:SOT-23-6 -> Li_Ion_LE:SOT-23-6
- U2: footprint Li-ion:SOT65P280X95-8N -> Li_Ion_LE:SOT65P280X95-8N
- U3: footprint Li-ion:MCP73833 -> Li_Ion_LE:MCP73833
- U4: footprint Li-ion:PAM2423AECADJR -> Li_Ion_LE:PAM2423AECADJR
- W1, W2, W3, W4, W5, W6, W7, W8: footprint Li-ion:Pad_3.0-5.0_w_TH -> Li_Ion_LE:Pad_3.0-5.0_w_TH
Other:
- note added: "Additional Features"

Commit message: Updates after first build, intermediate check in
Parts:
- added FID4: Fiducial, Fiducial_LE:Fiducial_1mm_Mask2mm, symbol Mechanical_LE:Fiducial
- added H1, H2, H3, H4: MountingHole, MountingHole:MountingHole_2.2mm_M2, symbol Mechanical:MountingHole
- C1: footprint Frequently_Used_LE:0805_2012Metric_HandSolder -> Frequently_Used_LE:0603_1608Metric; Description 0.1µF ±20% 50V Ceramic Capacitor X7R 0805 (2012 Metric) -> 0.1µF ±20% 50V Ceramic Capacitor; Manufacturer Part No. CL21B104MBCNNNC -> CL10B104JB8NNNC; Source 2 (none) -> Mouser; Source 2 Part No. (none) -> 187-CL10B104JB8NNNC; Source Part No. 1276-2450-1-ND -> -
- C10, C4: footprint Frequently_Used_LE:0805_2012Metric_HandSolder -> Frequently_Used_LE:0603_1608Metric; Description 10µF ±10% 6.3V Ceramic Capacitor X5R 0805 (2012 Metric) -> 10µF ±10% 10V Ceramic Capacitor X5R; Manufacturer Part No. CL21A106KQCLRNC -> CL10A106KP8NQSC; Source 2 (none) -> Mouser; Source 2 Part No. (none) -> 187-CL10A106KP8NQSC; Source Part No. 1276-2405-1-ND -> -
- C11, C3: Source 2 (none) -> Mouser; Source 2 Part No. (none) -> 232-25TLV470M10X10.5
- C2, C8: footprint Frequently_Used_LE:0805_2012Metric_HandSolder -> Frequently_Used_LE:0603_1608Metric; Description 22µF ±10% 6.3V Ceramic Capacitor X5R 0805 (2012 Metric) -> 22µF ±20% 6.3V Ceramic Capacitor X5R; Manufacturer Part No. CL21A226KQCLRNC -> CL10A226MQ8NRNE; Source 2 (none) -> Mouser; Source 2 Part No. (none) -> 187-CL10A226MQ8NRNE; Source Part No. 1276-6687-1-ND -> -
- C5: footprint Frequently_Used_LE:0805_2012Metric_HandSolder -> Frequently_Used_LE:0603_1608Metric; Description 2200pF ±10% 50V Ceramic Capacitor X7R 0805 (2012 Metric) -> 2200pF ±10% 50V Ceramic Capacitor X7R; Manufacturer Part No. CL21B222KBANNNC -> CL10B222KB8NFNC; Source 2 (none) -> Mouser; Source 2 Part No. (none) -> 187-CL10B222KB8NFNC; Source Part No. 1276-1171-1-ND -> -
- C6: footprint Frequently_Used_LE:0805_2012Metric_HandSolder -> Frequently_Used_LE:0603_1608Metric; Description 1µF ±10% 16V Ceramic Capacitor X7R 0805 (2012 Metric) -> 1µF ±10% 25V Ceramic Capacitor X7R; Manufacturer Part No. CL21B105KOFNNWE -> CL10A105KA8NFNC; Source 2 (none) -> Mouser; Source 2 Part No. (none) -> 187-CL10A105KA8NFNC; Source Part No. 1276-2931-1-ND -> -
- C7: footprint Frequently_Used_LE:0805_2012Metric_HandSolder -> Frequently_Used_LE:0603_1608Metric; Description 47pF ±5% 50V Ceramic Capacitor C0G, NP0 0805 (2012 Metric) -> 47pF ±5% 50V Ceramic Capacitor C0G, NP0; Manufacturer Part No. CL21C470JBANNNC -> CL10C470JB81PNC; Source 2 (none) -> Mouser; Source 2 Part No. (none) -> 187-CL10C470JB81PNC; Source Part No. 1276-1156-1-ND -> -
- C9: footprint Frequently_Used_LE:0805_2012Metric_HandSolder -> Frequently_Used_LE:0603_1608Metric; Description 10000pF ±10% 50V Ceramic Capacitor X7R 0805 (2012 Metric) -> 10000pF ±10% 50V Ceramic Capacitor X7R; Manufacturer Part No. CL21B103KBANNNC -> CL10B103KB8NNNL; Source 2 (none) -> Mouser; Source 2 Part No. (none) -> 187-CL10B103KB8NNNL; Source Part No. 1276-1015-1-ND -> -
- D1: Source 2 (none) -> Mouser; Source 2 Part No. (none) -> 863-NTS12120EMFST1G
- FID1, FID2, FID3: Source 2 (none) -> Mouser; Source 2 Part No. (none) -> None
- J1: footprint Connector_LE:GCT_USB4110-GF-A -> Connector_LE:GCT_USB4125-GF-A_REVA; symbol Connector_LE:USB_C_Plug_USB2.0 -> Connector_LE:USB_C_Plug_Power; Description USB-C 2.0 Female SMD Connector -> USB-C Power Female SMD Connector; Manufacturer Part No. USB4110-GF-A -> USB4125-GF-A; Source 2 (none) -> Mouser; Source 2 Part No. (none) -> 640-USB4125-GF-A; Source Part No. 2073-USB4110-GF-A-1-ND -> 2073-USB4125-GF-ACT-ND
- L1: Source 2 (none) -> Mouser; Source 2 Part No. (none) -> 875-MGV10046R8M-10
- LD1, LD2: footprint Li_Ion_LE:LED_0805_2012Metric_HandSolder -> Frequently_Used_LE:LED_0805_2012Metric; Description Green 570nm LED Indication - Discrete 2V 0805 (2012 Metric) -> Green 570nm LED Indication - Discrete 2V; Source 2 (none) -> Mouser; Source 2 Part No. (none) -> 710-150080VS75000
- LD3, LD4: footprint Li_Ion_LE:LED_0805_2012Metric_HandSolder -> Frequently_Used_LE:LED_0805_2012Metric; Description Red 625nm LED Indication - Discrete 2V 0805 (2012 Metric) -> Red 625nm LED Indication - Discrete 2V; Source 2 (none) -> Mouser; Source 2 Part No. (none) -> 710-150080RS75000
- R1: footprint Frequently_Used_LE:0805_2012Metric_HandSolder -> Frequently_Used_LE:0603_1608Metric; Description 330 Ohms ±1% 0.25W, 1/4W Chip Resistor 1206 (3216 Metric) -> 330 Ohms ±1% 0.25W, 1/4W Chip Resistor; Manufacturer Name KOA Speer Electronics, Inc. -> ROHM Semiconductor; Manufacturer Part No. RK73H2ATTD3300F -> ESR03EZPF3300; Source 2 (none) -> Mouser; Source 2 Part No. (none) -> 755-ESR03EZPF3300; Source Part No. 2019-RK73H2ATTD3300FCT-ND -> -
- R10: footprint Frequently_Used_LE:0805_2012Metric_HandSolder -> Frequently_Used_LE:0603_1608Metric; Description 30 kOhms ±1% 0.25W, 1/4W Chip Resistor 1206 (3216 Metric) -> 30 kOhms ±1% 0.25W, 1/4W Chip Resistor; Manufacturer Name KOA Speer Electronics, Inc. -> ROHM Semiconductor; Manufacturer Part No. RK73H2ATTD3002F -> ESR03EZPF3002; Source 2 (none) -> Mouser; Source 2 Part No. (none) -> 755-ESR03EZPF3002; Source Part No. 2019-RK73H2ATTD3002FCT-ND -> -
- R11: footprint Frequently_Used_LE:0805_2012Metric_HandSolder -> Frequently_Used_LE:0603_1608Metric; Description 10 kOhms ±1% 0.25W, 1/4W Chip Resistor 1206 (3216 Metric) -> 10 kOhms ±1% 0.25W, 1/4W Chip Resistor; Manufacturer Name KOA Speer Electronics, Inc. -> ROHM Semiconductor; Manufacturer Part No. RK73H2ATTD1002F -> ESR03EZPF1002; Source 2 (none) -> Mouser; Source 2 Part No. (none) -> 755-ESR03EZPF1002; Source Part No. 2019-RK73H2ATTD1002FCT-ND -> -
- R12, R3, R4, R5, R6: footprint Frequently_Used_LE:0805_2012Metric_HandSolder -> Frequently_Used_LE:0603_1608Metric; Description 1 kOhms ±1% 0.25W, 1/4W Chip Resistor 1206 (3216 Metric) -> 1 kOhms ±1% 0.25W, 1/4W Chip Resistor; Manufacturer Name KOA Speer Electronics, Inc. -> ROHM Semiconductor; Manufacturer Part No. RK73H2ATTD1001F -> ESR03EZPF1001; Source 2 (none) -> Mouser; Source 2 Part No. (none) -> 755-ESR03EZPF1001; Source Part No. 2019-RK73H2ATTD1001FCT-ND -> -
- R2: footprint Frequently_Used_LE:0805_2012Metric_HandSolder -> Frequently_Used_LE:0603_1608Metric; Description 2.7 kOhms ±1% 0.25W, 1/4W Chip Resistor 1206 (3216 Metric) -> 2.7 kOhms ±1% 0.25W, 1/4W Chip Resistor; Manufacturer Name KOA Speer Electronics, Inc. -> ROHM Semiconductor; Manufacturer Part No. RK73H2ATTD2701F -> ESR03EZPF2701; Source 2 (none) -> Mouser; Source 2 Part No. (none) -> 755-ESR03EZPF2701; Source Part No. 2019-RK73H2ATTD2701FCT-ND -> -
- R7: footprint Frequently_Used_LE:0805_2012Metric_HandSolder -> Frequently_Used_LE:0603_1608Metric; Description 1.54 kOhms ±1% 0.25W, 1/4W Chip Resistor 1206 (3216 Metric) -> 1.5 kOhms ±1% 0.25W, 1/4W Chip Resistor; Manufacturer Name KOA Speer Electronics, Inc. -> ROHM Semiconductor; Manufacturer Part No. RK73H2ATTD1541F -> ESR03EZPF1501; Source 2 (none) -> Mouser; Source 2 Part No. (none) -> 755-ESR03EZPF1501; Source Part No. 2019-RK73H2ATTD1541FCT-ND -> -
- R8: footprint Frequently_Used_LE:0805_2012Metric_HandSolder -> Frequently_Used_LE:0603_1608Metric; Description 69.8 kOhms ±1% 0.25W, 1/4W Chip Resistor 1206 (3216 Metric) -> 68 kOhms ±1% 0.25W, 1/4W Chip Resistor; Manufacturer Name KOA Speer Electronics, Inc. -> ROHM Semiconductor; Manufacturer Part No. RK73H2ATTD6982F -> ESR03EZPF6802; Source 2 (none) -> Mouser; Source 2 Part No. (none) -> 755-ESR03EZPF6802; Source Part No. 2019-RK73H2ATTD6982FCT-ND -> -
- R9: footprint Frequently_Used_LE:0805_2012Metric_HandSolder -> Frequently_Used_LE:0603_1608Metric; Description 51 kOhms ±1% 0.25W, 1/4W Chip Resistor 1206 (3216 Metric) -> 51 kOhms ±1% 0.25W, 1/4W Chip Resistor; Manufacturer Name KOA Speer Electronics, Inc. -> ROHM Semiconductor; Manufacturer Part No. RK73H2ATTD5102F -> ESR03EZPF5102; Source 2 (none) -> Mouser; Source 2 Part No. (none) -> 755-ESR03EZPF5102; Source Part No. 2019-RK73H2ATTD5102FCT-ND -> -
- SW1: Source 2 (none) -> Mouser
- TH1: footprint Frequently_Used_LE:0805_2012Metric_HandSolder -> Frequently_Used_LE:0603_1608Metric; Manufacturer Part No. NTCG203NH103JT1 -> NTCG163JH103JT; Source 2 (none) -> Mouser; Source 2 Part No. (none) -> 810-NTCG163JH103JT; Source Part No. 445-175460-1-ND -> -
- U1: Source 2 (none) -> Mouser; Source 2 Part No. (none) -> 621-AP9101CK6-AYTRG1
- U2: Source 2 (none) -> Mouser; Source 2 Part No. (none) -> 863-ECH8695R-TL-W
- U3: Source 2 (none) -> Mouser; Source 2 Part No. (none) -> 579-MCP73833T-AMI/UN
- U4: Source 2 (none) -> Mouser; Source 2 Part No. (none) -> 621-PAM2423AECADJR
- W1, W2, W3, W4, W5, W6, W7, W8: value 2.5x5.0 -> 2.0x3.25; footprint Li_Ion_LE:Pad_3.0-5.0_w_TH -> Li_Ion_LE:Pad_2.0-3.25_w_TH; Source 2 (none) -> Mouser; Source 2 Part No. (none) -> None
Connections:
- no-connect marks 16 -> 10
Other:
- moved on the sheet: FID1, FID2, FID3

Commit message: Version 1.1 updates
Parts:
- added Q1: BUK6D30-40E, Li_Ion_LE:BUK6D3040EX, symbol Li_Ion_LE:BUK6D30-40E
- added R13: 330, Frequently_Used_LE:0603_1608Metric, symbol Frequently_Used_LE:R
- added R14: 10k, Frequently_Used_LE:0603_1608Metric, symbol Frequently_Used_LE:R
- C11, C3: footprint Li_Ion_LE:25TLV470M10X10.5 -> Li_Ion_LE:CP_Elec_10x10.5
- H1, H2, H3, H4: Description (none) -> M2 mounting hole; Manufacturer Name (none) -> None; Manufacturer Part No. (none) -> None; Source 2 Part No. (none) -> None; Source Part No. (none) -> None
- J1: footprint Connector_LE:GCT_USB4125-GF-A_REVA -> Connector_LE:GCT_USB4110-GF-A; symbol Connector_LE:USB_C_Plug_Power -> Connector_LE:USB_C_Plug_USB2.0; Manufacturer Part No. USB4125-GF-A -> USB4110-GF-A; Source 2 Part No. 640-USB4125-GF-A -> 640-USB4110-GF-A; Source Part No. 2073-USB4125-GF-ACT-ND -> 2073-USB4110-GF-A-1-ND
- SW1: footprint Li_Ion_LE:GF1230054 -> Button_Switch_LE:CL-SB-22A_Edge; Description Slide Switch SPST Through Hole 8.5A 125V -> Slide Switch DPDT Surface Mount, Right Angle; Manufacturer Name CW Industries -> Nidec Copal Electronics; Manufacturer Part No. GF-123-0054 -> CL-SB-22A-11T; Source 2 Part No. (none) -> 229-CL-SB-22A-11T; Source Part No. CWI333-ND -> 563-1340-1-ND
- renumbered FID1 to F1, FID2 to F2, FID3 to F3, FID4 to F4
Connections:
- net labels added: BGND
- wire segments 178 -> 176
- no-connect marks 10 -> 16
Other:
- note added: "Switch"
- moved on the sheet: C1, C10, C11, C2, C3, C4, C5, C6, C7, C8, C9, D1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

Commit message: Version 1.1 updates
Version 1.1 updates
Parts:
- SW1: value SW_SPST -> SW_DPST; symbol Frequently_Used_LE:SW_SPST -> Button_Switch_LE:CL-SB-22A
- W3, W4: value 2.0x3.25 -> 1.5x2.5; footprint Li_Ion_LE:Pad_2.0-3.25_w_TH -> Li_Ion_LE:Pad_1.5-2.5_w_TH
Connections:
- wire segments 176 -> 174
- no-connect marks 16 -> 17
Other:
- moved on the sheet: R13, R14, W3, W4
Changed lines of the file:
@@
 	1    0    0    -1
 $EndComp
-Text Label 7550 1650 0    50   ~ 0
+Text Label 7500 1650 0    50   ~ 0
 BATT+
 $Comp
-L Frequently_Used_LE:TestPoint_1 W3
-U 1 1 5EC3644F
-P 7950 1450
-F 0 "W3" V 7850 1500 59  0000 L CNN
-F 1 "2.0x3.25" V 8000 1500 59  0000 L TNN
-F 2 "Li_Ion_LE:Pad_2.0-3.25_w_TH" H 7950 1450 50  0001 C CNN
-F 3 "None" H 7950 1450 50  0001 C CNN
-F 4 "Wire solder point" H 7950 1450 50  0001 C CNN "Description"
-F 5 "None" H 7950 1450 50  0001 C CNN "Source Part No."
-F 6 "None" H 7950 1450 50  0001 C CNN "Manufacturer Part No."
-F 7 "None" H 7950 1450 50  0001 C CNN "Manufacturer Name"
-F 8 "None" H 7950 1450 50  0001 C CNN "Source"
-F 9 "Mouser" H 7950 1450 50  0001 C CNN "Source 2"
-F 10 "None" H 7950 1450 50  0001 C CNN "Source 2 Part No."
-	1    7950 1450
-	1    0    0    -1
-$EndComp
-$Comp
-L Frequently_Used_LE:TestPoint_1 W4
-U 1 1 5EC17D57
-P 8350 1450
-F 0 "W4" V 8250 1500 59  0000 L CNN
-F 1 "2.0x3.25" V 8400 1500 59  0000 L TNN
-F 2 "Li_Ion_LE:Pad_2.0-3.25_w_TH" H 8350 1450 50  0001 C CNN
-F 3 "None" H 8350 1450 50  0001 C CNN
-F 4 "Wire solder point" H 8350 1450 50  0001 C CNN "Description"
-F 5 "None" H 8350 1450 50  0001 C CNN "Source Part No."
-F 6 "None" H 8350 1450 50  0001 C CNN "Manufacturer Part No."
-F 7 "None" H 8350 1450 50  0001 C CNN "Manufacturer Name"
-F 8 "None" H 8350 1450 50  0001 C CNN "Source"
-F 9 "Mouser" H 8350 1450 50  0001 C CNN "Source 2"
-F 10 "None" H 8350 1450 50  0001 C CNN "Source 2 Part No."
-	1    8350 1450
-	1    0    0    -1
-$EndComp
-$Comp
-L Frequently_Used_LE:SW_SPST SW1
+L Button_Switch_LE:CL-SB-22A SW1
 U 1 1 5EE83AA5
 P 8150 1650
-F 0 "SW1" H 8150 1800 50  0000 C CNN
-F 1 "SW_SPST" H 8150 1900 50  0000 C CNN
+F 0 "SW1" H 8050 1500 50  0000 C CNN
+F 1 "SW_DPST" H 8140 1430 50  0000 C CNN
 F 2 "Button_Switch_LE:CL-SB-22A_Edge" H 8150 1650 50  0001 C CNN
 F 3 "https://www.nidec-copal-electronics.com/e/catalog/switch/cl-sb.pdf" H 8150 1650 50  0001 C CNN
@@
 F 10 "229-CL-SB-22A-11T" H 8150 1650 50  0001 C CNN "Source 2 Part No."
 	1    8150 1650
-	-1   0    0    1
+	1    0    0    -1
 $EndComp
 $Comp
 L Frequently_Used_LE:R R14
 U 1 1 60844507
-P 9500 1400
-F 0 "R14" H 9550 1450 59  0000 L CNN
-F 1 "10k" H 9550 1350 59  0000 L CNN
-F 2 "Frequently_Used_LE:0603_1608Metric" H 9500 1400 50  0001 C CNN
-F 3 "https://www.mouser.com/datasheet/2/348/esr_e-1139161.pdf" H 9500 1400 50  0001 C CNN
-F 4 "10 kOhms ±1% 0.25W, 1/4W Chip Resistor" H 9500 1400 50  0001 C CNN "Description"
-F 5 "-" H 9500 1400 50  0001 C CNN "Source Part No."
-F 6 "ESR03EZPF1002" H 9500 1400 50  0001 C CNN "Manufacturer Part No."
-F 7 "ROHM Semiconductor" H 9500 1400 50  0001 C CNN "Manufacturer Name"
-F 8 "Digikey" H 9500 1400 50  0001 C CNN "Source"
-F 9 "Mouser" H 9500 1400 50  0001 C CNN "Source 2"
-F 10 "755-ESR03EZPF1002" H 9500 1400 50  0001 C CNN "Source 2 Part No."
-	1    9500 1400
+P 9470 1400
+F 0 "R14" H 9520 1450 59  0000 L CNN
+F 1 "10k" H 9520 1350 59  0000 L CNN
+F 2 "Frequently_Used_LE:0603_1608Metric" H 9470 1400 50  0001 C CNN
+F 3 "https://www.mouser.com/datasheet/2/348/esr_e-1139161.pdf" H 9470 1400 50  0001 C CNN
+F 4 "10 kOhms ±1% 0.25W, 1/4W Chip Resistor" H 9470 1400 50  0001 C CNN "Description"
+F 5 "-" H 9470 1400 50  0001 C CNN "Source Part No."
+F 6 "ESR03EZPF1002" H 9470 1400 50  0001 C CNN "Manufacturer Part No."
+F 7 "ROHM Semiconductor" H 9470 1400 50  0001 C CNN "Manufacturer Name"
+F 8 "Digikey" H 9470 1400 50  0001 C CNN "Source"
+F 9 "Mouser" H 9470 1400 50  0001 C CNN "Source 2"
+F 10 "755-ESR03EZPF1002" H 9470 1400 50  0001 C CNN "Source 2 Part No."
+	1    9470 1400
 	1    0    0    -1
 $EndComp
 Text Label 8600 1150 0    50   ~ 0
 BGND
-Wire Wire Line
-	9350 1150 9500 1150
 Wire Wire Line
 	9850 1150 9850 1250
@@
 	9150 1450 9150 1650
 Wire Wire Line
-	9150 1650 8950 1650
+	9150 1650 9060 1650
 Wire Wire Line
-	8650 1650 8450 1650
+	8760 1650 8540 1650
 Wire Wire Line
-	8350 1450 8350 1550
+	8540 1520 8540 1650
 Wire Wire Line
-	8350 1550 8450 1550
-Wire Wire Line
-	8450 1550 8450 1650
-Connection ~ 8450 1650
-Wire Wire Line
-	8450 1650 8350 1650
+	8370 1750 8370 1650
 Wire Wire Line
 	7950 1650 7850 1650
 Wire Wire Line
-	7950 1450 7950 1550
-Wire Wire Line
-	7950 1550 7850 1550
-Wire Wire Line
-	7850 1550 7850 1650
+	7850 1520 7850 1650
 Connection ~ 7850 1650
 Wire Wire Line
-	7850 1650 7550 1650
+	7850 1650 7500 1650
 Wire Wire Line
-	9500 1250 9500 1150
-Connection ~ 9500 1150
+	9470 1550 9470 1650
 Wire Wire Line
-	9500 1150 9850 1150
-Wire Wire Line
-	9500 1550 9500 1650
-Wire Wire Line
-	9500 1650 9150 1650
+	9470 1650 9150 1650
 Connection ~ 9150 1650
 $Comp
 L Frequently_Used_LE:R R13
 U 1 1 6095E97E
-P 8800 1650
-F 0 "R13" V 8700 1550 59  0000 L CNN
-F 1 "330" V 8900 1550 59  0000 L CNN
-F 2 "Frequently_Used_LE:0603_1608Metric" H 8800 1650 50  0001 C CNN
-F 3 "https://www.mouser.com/datasheet/2/348/esr_e-1139161.pdf" H 8800 1650 50  0001 C CNN
-F 4 "330 Ohms ±1% 0.25W, 1/4W Chip Resistor" H 8800 1650 50  0001 C CNN "Description"
-F 5 "-" H 8800 1650 50  0001 C CNN "Source Part No."
-F 6 "ESR03EZPF3300" H 8800 1650 50  0001 C CNN "Manufacturer Part No."
-F 7 "ROHM Semiconductor" H 8800 1650 50  0001 C CNN "Manufacturer Name"
-F 8 "Digikey" H 8800 1650 50  0001 C CNN "Source"
-F 9 "Mouser" H 8800 1650 50  0001 C CNN "Source 2"
-F 10 "755-ESR03EZPF3300" H 8800 1650 50  0001 C CNN "Source 2 Part No."
-	1    8800 1650
+P 8910 1650
+F 0 "R13" V 8810 1550 59  0000 L CNN
+F 1 "330" V 9010 1550 59  0000 L CNN
+F 2 "Frequently_Used_LE:0603_1608Metric" H 8910 1650 50  0001 C CNN
+F 3 "https://www.mouser.com/datasheet/2/348/esr_e-1139161.pdf" H 8910 1650 50  0001 C CNN
+F 4 "330 Ohms ±1% 0.25W, 1/4W Chip Resistor" H 8910 1650 50  0001 C CNN "Description"
+F 5 "-" H 8910 1650 50  0001 C CNN "Source Part No."
+F 6 "ESR03EZPF3300" H 8910 1650 50  0001 C CNN "Manufacturer Part No."
+F 7 "ROHM Semiconductor" H 8910 1650 50  0001 C CNN "Manufacturer Name"
+F 8 "Digikey" H 8910 1650 50  0001 C CNN "Source"
+F 9 "Mouser" H 8910 1650 50  0001 C CNN "Source 2"
+F 10 "755-ESR03EZPF3300" H 8910 1650 50  0001 C CNN "Source 2 Part No."
+	1    8910 1650
 	0    1    1    0
 $EndComp
@@
 U 1 1 E0548A51
 P 8125 3350
-F 0 "D1" H 8025 3550 59  0000 L TNN
+F 0 "D1" H 8060 3490 59  0000 L TNN
 F 1 "NTS12120EMFST1G" H 8125 3200 59  0000 C CNN
 F 2 "Li_Ion_LE:NTS12120EMFST1G" H 8125 3350 50  0001 C CNN
@@
 Wire Wire Line
 	8275 3350 8475 3350
+Wire Wire Line
+	8350 1750 8370 1750
+Connection ~ 8540 1650
+Wire Wire Line
+	8540 1650 8370 1650
+$Comp
+L Frequently_Used_LE:TestPoint_1 W3
+U 1 1 5EC3644F
+P 7850 1520
+F 0 "W3" H 7660 1770 59  0000 L CNN
+F 1 "1.5x2.5" H 7660 1710 59  0000 L TNN
+F 2 "Li_Ion_LE:Pad_1.5-2.5_w_TH" H 7850 1520 50  0001 C CNN
+F 3 "None" H 7850 1520 50  0001 C CNN
+F 4 "Wire solder point" H 7850 1520 50  0001 C CNN "Description"
+F 5 "None" H 7850 1520 50  0001 C CNN "Source Part No."
+F 6 "None" H 7850 1520 50  0001 C CNN "Manufacturer Part No."
+F 7 "None" H 7850 1520 50  0001 C CNN "Manufacturer Name"
+F 8 "None" H 7850 1520 50  0001 C CNN "Source"
+F 9 "Mouser" H 7850 1520 50  0001 C CNN "Source 2"
+F 10 "None" H 7850 1520 50  0001 C CNN "Source 2 Part No."
+	1    7850 1520
+	1    0    0    -1
+$EndComp
+$Comp
+L Frequently_Used_LE:TestPoint_1 W4
+U 1 1 5EC17D57
+P 8540 1520
+F 0 "W4" H 8340 1780 59  0000 L CNN
+F 1 "1.5x2.5" H 8340 1710 59  0000 L TNN
+F 2 "Li_Ion_LE:Pad_1.5-2.5_w_TH" H 8540 1520 50  0001 C CNN
+F 3 "None" H 8540 1520 50  0001 C CNN
+F 4 "Wire solder point" H 8540 1520 50  0001 C CNN "Description"
+F 5 "None" H 8540 1520 50  0001 C CNN "Source Part No."
+F 6 "None" H 8540 1520 50  0001 C CNN "Manufacturer Part No."
+F 7 "None" H 8540 1520 50  0001 C CNN "Manufacturer Name"
+F 8 "None" H 8540 1520 50  0001 C CNN "Source"
+F 9 "Mouser" H 8540 1520 50  0001 C CNN "Source 2"
+F 10 "None" H 8540 1520 50  0001 C CNN "Source 2 Part No."
+	1    8540 1520
+	1    0    0    -1
+$EndComp
+Wire Wire Line
+	9350 1150 9470 1150
+Wire Wire Line
+	9470 1250 9470 1150
+Connection ~ 9470 1150
+Wire Wire Line
+	9470 1150 9850 1150
+NoConn ~ 8350 1550
 $EndSCHEMATC

Commit message: Near complete version 1.1.0
Other:
- moved on the sheet: SW1
Changed lines of the file:
@@
 F 1 "USB_C_FEMALE" H 950 7300 70  0000 L CNN
 F 2 "Connector_LE:GCT_USB4110-GF-A" H 1300 6600 50  0001 C CNN
-F 3 "https://gct.co/files/drawings/usb4125.pdf" H 1300 6600 50  0001 C CNN
+F 3 "https://www.mouser.com/datasheet/2/837/USB4110-1948945.pdf" H 1300 6600 50  0001 C CNN
 F 4 "USB-C Power Female SMD Connector" H 1300 6600 50  0001 C CNN "Description"
 F 5 "2073-USB4110-GF-A-1-ND" H 1300 6600 50  0001 C CNN "Source Part No."
@@
 L Button_Switch_LE:CL-SB-22A SW1
 U 1 1 5EE83AA5
-P 8150 1650
-F 0 "SW1" H 8050 1500 50  0000 C CNN
-F 1 "SW_DPST" H 8140 1430 50  0000 C CNN
-F 2 "Button_Switch_LE:CL-SB-22A_Edge" H 8150 1650 50  0001 C CNN
-F 3 "https://www.nidec-copal-electronics.com/e/catalog/switch/cl-sb.pdf" H 8150 1650 50  0001 C CNN
-F 4 "Slide Switch DPDT Surface Mount, Right Angle" H 8150 1650 50  0001 C CNN "Description"
-F 5 "563-1340-1-ND" H 8150 1650 50  0001 C CNN "Source Part No."
-F 6 "CL-SB-22A-11T" H 8150 1650 50  0001 C CNN "Manufacturer Part No."
-F 7 "Nidec Copal Electronics" H 8150 1650 50  0001 C CNN "Manufacturer Name"
-F 8 "Digikey" H 8150 1650 50  0001 C CNN "Source"
-F 9 "Mouser" H 8150 1650 50  0001 C CNN "Source 2"
-F 10 "229-CL-SB-22A-11T" H 8150 1650 50  0001 C CNN "Source 2 Part No."
-	1    8150 1650
-	1    0    0    -1
+P 8150 1750
+F 0 "SW1" H 8050 1600 50  0000 C CNN
+F 1 "SW_DPST" H 8140 1530 50  0000 C CNN
+F 2 "Button_Switch_LE:CL-SB-22A_Edge" H 8150 1750 50  0001 C CNN
+F 3 "https://www.nidec-copal-electronics.com/e/catalog/switch/cl-sb.pdf" H 8150 1750 50  0001 C CNN
+F 4 "Slide Switch DPDT Surface Mount, Right Angle" H 8150 1750 50  0001 C CNN "Description"
+F 5 "563-1340-1-ND" H 8150 1750 50  0001 C CNN "Source Part No."
+F 6 "CL-SB-22A-11T" H 8150 1750 50  0001 C CNN "Manufacturer Part No."
+F 7 "Nidec Copal Electronics" H 8150 1750 50  0001 C CNN "Manufacturer Name"
+F 8 "Digikey" H 8150 1750 50  0001 C CNN "Source"
+F 9 "Mouser" H 8150 1750 50  0001 C CNN "Source 2"
+F 10 "229-CL-SB-22A-11T" H 8150 1750 50  0001 C CNN "Source 2 Part No."
+	1    8150 1750
+	-1   0    0    1
 $EndComp
 $Comp
@@
 Wire Wire Line
 	9470 1150 9850 1150
-NoConn ~ 8350 1550
+NoConn ~ 7950 1850
 $EndSCHEMATC
