File: Li-ion 5.5A Boost 1A Charge Protect/Li-ion 5.5A Boost 1A Charge Protect.sch (KiCad schematic (older format))
At the start: 20 parts, among them J1 USB_C_FEMALE

Commit message: House keeping updates.
Parts:
- H1, H2, H3, H4: symbol Mechanical:MountingHole -> Mechanical_LE:MountingHole
Changed lines of the file:
@@
 $EndComp
 $Comp
-L Mechanical:MountingHole H1
+L Mechanical_LE:MountingHole H1
 U 1 1 608288AB
 P 2745 6850
@@
 $EndComp
 $Comp
-L Mechanical:MountingHole H2
+L Mechanical_LE:MountingHole H2
 U 1 1 6084B9CC
 P 3495 6850
@@
 $EndComp
 $Comp
-L Mechanical:MountingHole H3
+L Mechanical_LE:MountingHole H3
 U 1 1 6084C007
 P 2745 7100
@@
 $EndComp
 $Comp
-L Mechanical:MountingHole H4
+L Mechanical_LE:MountingHole H4
 U 1 1 6084C489
 P 3495 7100
