File: Li-ion 5.5A Boost 1A Charge Protect/Li-ion 5.5A Boost 1A Charge Protect.kicad_pcb (KiCad board)
At the start: 2 copper layers, 51.5 x 32 mm, 58 parts, among them J1 USB_C_FEMALE, Q1 BUK6D30-40E, SW1 SW_DPST, U1 AP9101CK6, U2 ECH8695R-TL-W, U3 MCP73833T, U4 PAM2423AECADJR

Commit message: Update version text
Other:
- board text added: "V1.1.1"
- board text removed: "V1.1.0"
Changed lines of the file:
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@@
-(kicad_pcb (version 20171130) (host pcbnew "(5.1.9)-1")
+(kicad_pcb (version 20171130) (host pcbnew "(5.1.5)-3")
   (general
     (thickness 1.6)
@@
   (layers
     (0 F.Cu signal)
-    (31 B.Cu signal hide)
+    (31 B.Cu signal)
     (32 B.Adhes user hide)
     (33 F.Adhes user hide)
-    (34 B.Paste user hide)
-    (35 F.Paste user)
-    (36 B.SilkS user hide)
-    (37 F.SilkS user)
-    (38 B.Mask user hide)
-    (39 F.Mask user)
+    (34 B.Paste user)
+    (35 F.Paste user hide)
+    (36 B.SilkS user)
+    (37 F.SilkS user hide)
+    (38 B.Mask user)
+    (39 F.Mask user hide)
     (40 Dwgs.User user hide)
     (41 Cmts.User user hide)
@@
     (effects (font (size 1.5 1.5) (thickness 0.3)) (justify left mirror))
   )
-  (gr_text V1.1.0 (at 151.19 90.72) (layer B.SilkS)
+  (gr_text V1.1.1 (at 151.19 90.72) (layer B.SilkS)
     (effects (font (size 1.5 1.5) (thickness 0.3)) (justify left mirror))
   )
